File: F22 V2 Wiring Schematic-backups/F22 V2 Wiring Schematic-2022-10-19_180049 2/FuseBox.kicad_sch (KiCad schematic)
At the start: 2 parts

Commit message: Test Oct20
Other:
- removed sheet Coil Overview
- moved on the sheet: U?
