File: F22 V2 Wiring Schematic-backups/F22 V2 Wiring Schematic-2022-10-12_180330/F22 V2 Wiring Schematic-backups/F22 V2 Wiring Schematic-2022-10-20_095645/DTM-Dash.kicad_sch (KiCad schematic)
At the start: 10 parts

Commit message: Idk
Connections:
- new net: F?.2, U?., U?.
- new net: D?.1 (A), U?., U?.
- now unconnected: U?., U?.
