File: F22 V2 Wiring Schematic-backups/F22 V2 Wiring Schematic-2022-10-12_180330/F22 V2 Wiring Schematic-backups/F22 V2 Wiring Schematic-2022-10-20_095645/FuseBox.kicad_sch (KiCad schematic)
At the start: 2 parts

Commit message: Idk
Other:
- removed sheet Engine Overview
- moved on the sheet: U?
