File: ECU-Main-Loom.kicad_sch (KiCad schematic)
At the start: 1 part

Commit message: Create new top level
Parts:
- U?: value ECU -> (none)
Changed lines of the file:
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@@
     (effects (font (size 1.27 1.27)) (justify left bottom))
+  )
+  (global_label "CANH" (shape input) (at 52.324 54.102 0) (fields_autoplaced)
+    (effects (font (size 1.27 1.27)) (justify left))
+    (property "Intersheet References" "${INTERSHEET_REFS}" (id 0) (at 59.7566 54.0226 0)
+      (effects (font (size 1.27 1.27)) (justify left) hide)
+    )
   )
   (symbol (lib_id "Ty lib:ECU") (at 86.106 50.8 0) (unit 1)
@@
       (effects (font (size 1.27 1.27)) (justify left) hide)
     )
-    (property "Value" "ECU" (id 1) (at 155.956 55.3719 0)
+    (property "Value" "" (id 1) (at 155.956 55.3719 0)
       (effects (font (size 1.27 1.27)) (justify left) hide)
     )

Commit message: HUGE TOP LEVEL
Parts:
- U?: value (none) -> ECU
Changed lines of the file:
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@@
       (effects (font (size 1.27 1.27)) (justify left) hide)
     )
-    (property "Value" "" (id 1) (at 155.956 55.3719 0)
+    (property "Value" "ECU" (id 1) (at 155.956 55.3719 0)
       (effects (font (size 1.27 1.27)) (justify left) hide)
     )
