File: Coil_Overview.kicad_sch (KiCad schematic)
At the start: 5 parts

Commit message: Create new top level
Parts:
- Coil?, INJ?: value L -> (none)
- U?: value 3 -> (none)
- U?: value ECU2 -> (none)
- U?: value 4 -> (none)
Changed lines of the file:
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@@
       (effects (font (size 1.27 1.27)) hide)
     )
-    (property "Value" "GNDREF" (id 1) (at 134.366 141.478 0)
+    (property "Value" "" (id 1) (at 134.366 141.478 0)
       (effects (font (size 1.27 1.27)) hide)
     )
@@
       (effects (font (size 1.27 1.27)) hide)
     )
-    (property "Value" "GND" (id 1) (at 164.338 65.532 0))
+    (property "Value" "" (id 1) (at 164.338 65.532 0))
     (property "Footprint" "" (id 2) (at 164.338 59.944 0)
       (effects (font (size 1.27 1.27)) hide)
@@
       (effects (font (size 1.27 1.27)) (justify left) hide)
     )
-    (property "Value" "3" (id 1) (at 143.002 46.99 0)
+    (property "Value" "" (id 1) (at 143.002 46.99 0)
       (effects (font (size 1.27 1.27)) (justify left) hide)
     )
@@
       (effects (font (size 1.27 1.27)) (justify left))
     )
-    (property "Value" "L" (id 1) (at 131.572 135.1279 0)
+    (property "Value" "" (id 1) (at 131.572 135.1279 0)
       (effects (font (size 1.27 1.27)) (justify left) hide)
     )
@@
       (effects (font (size 1.27 1.27)) (justify left) hide)
     )
-    (property "Value" "ECU2" (id 1) (at 104.648 64.6429 0)
+    (property "Value" "" (id 1) (at 104.648 64.6429 0)
       (effects (font (size 1.27 1.27)) (justify left) hide)
     )
@@
       (effects (font (size 1.27 1.27)) hide)
     )
-    (property "Value" "-12V" (id 1) (at 152.908 122.936 0)
+    (property "Value" "" (id 1) (at 152.908 122.936 0)
       (effects (font (size 1.27 1.27)) hide)
     )
@@
       (effects (font (size 1.27 1.27)) (justify left))
     )
-    (property "Value" "L" (id 1) (at 149.86 138.1759 0)
+    (property "Value" "" (id 1) (at 149.86 138.1759 0)
       (effects (font (size 1.27 1.27)) (justify left) hide)
     )
@@
       (effects (font (size 1.27 1.27)) hide)
     )
-    (property "Value" "GND" (id 1) (at 131.826 123.19 0))
+    (property "Value" "" (id 1) (at 131.826 123.19 0))
     (property "Footprint" "" (id 2) (at 131.826 117.602 0)
       (effects (font (size 1.27 1.27)) hide)
@@
       (effects (font (size 1.27 1.27)) (justify left) hide)
     )
-    (property "Value" "4" (id 1) (at 163.068 64.0079 0)
+    (property "Value" "" (id 1) (at 163.068 64.0079 0)
       (effects (font (size 1.27 1.27)) (justify left) hide)
     )

Commit message: HUGE TOP LEVEL
Parts:
- Coil?, INJ?: value (none) -> L
- U?: value (none) -> 3
- U?: value (none) -> ECU2
- U?: value (none) -> 4
Changed lines of the file:
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@@
       (effects (font (size 1.27 1.27)) hide)
     )
-    (property "Value" "" (id 1) (at 134.366 141.478 0)
+    (property "Value" "GNDREF" (id 1) (at 134.366 141.478 0)
       (effects (font (size 1.27 1.27)) hide)
     )
@@
       (effects (font (size 1.27 1.27)) hide)
     )
-    (property "Value" "" (id 1) (at 164.338 65.532 0))
+    (property "Value" "GND" (id 1) (at 164.338 65.532 0))
     (property "Footprint" "" (id 2) (at 164.338 59.944 0)
       (effects (font (size 1.27 1.27)) hide)
@@
       (effects (font (size 1.27 1.27)) (justify left) hide)
     )
-    (property "Value" "" (id 1) (at 143.002 46.99 0)
+    (property "Value" "3" (id 1) (at 143.002 46.99 0)
       (effects (font (size 1.27 1.27)) (justify left) hide)
     )
@@
       (effects (font (size 1.27 1.27)) (justify left))
     )
-    (property "Value" "" (id 1) (at 131.572 135.1279 0)
+    (property "Value" "L" (id 1) (at 131.572 135.1279 0)
       (effects (font (size 1.27 1.27)) (justify left) hide)
     )
@@
       (effects (font (size 1.27 1.27)) (justify left) hide)
     )
-    (property "Value" "" (id 1) (at 104.648 64.6429 0)
+    (property "Value" "ECU2" (id 1) (at 104.648 64.6429 0)
       (effects (font (size 1.27 1.27)) (justify left) hide)
     )
@@
       (effects (font (size 1.27 1.27)) hide)
     )
-    (property "Value" "" (id 1) (at 152.908 122.936 0)
+    (property "Value" "-12V" (id 1) (at 152.908 122.936 0)
       (effects (font (size 1.27 1.27)) hide)
     )
@@
       (effects (font (size 1.27 1.27)) (justify left))
     )
-    (property "Value" "" (id 1) (at 149.86 138.1759 0)
+    (property "Value" "L" (id 1) (at 149.86 138.1759 0)
       (effects (font (size 1.27 1.27)) (justify left) hide)
     )
@@
       (effects (font (size 1.27 1.27)) hide)
     )
-    (property "Value" "" (id 1) (at 131.826 123.19 0))
+    (property "Value" "GND" (id 1) (at 131.826 123.19 0))
     (property "Footprint" "" (id 2) (at 131.826 117.602 0)
       (effects (font (size 1.27 1.27)) hide)
@@
       (effects (font (size 1.27 1.27)) (justify left) hide)
     )
-    (property "Value" "" (id 1) (at 163.068 64.0079 0)
+    (property "Value" "4" (id 1) (at 163.068 64.0079 0)
       (effects (font (size 1.27 1.27)) (justify left) hide)
     )
