File: DTM-Dash.kicad_sch (KiCad schematic)
At the start: 7 parts

Commit message: Changes to DTM Dash
Parts:
- D?: value DIODE -> LED
- U?: value 15 V Switch -> Ignition Switch
- U?: value Brake Override -> Brake Over-travel
Connections:
- net 12 V Fused Perm renamed Fuse 1 Power
- net 19 V Signal renamed IGN Signal
- new net: D?.1 (A), U?., U?.
Changed lines of the file:
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@@
     (stroke (width 0) (type default) (color 0 0 0 0))
   )
-  (label "12 V Fused Perm" (at 82.042 88.392 0)
+  (label "Fuse 1 Power" (at 82.042 88.392 0)
     (effects (font (size 0.762 0.762)) (justify left bottom))
   )
@@
     (effects (font (size 0.762 0.762)) (justify left bottom))
   )
-  (label "19 V Signal" (at 86.106 78.232 0)
+  (label "IGN Signal" (at 86.106 78.232 0)
     (effects (font (size 0.762 0.762)) (justify left bottom))
   )
@@
       (effects (font (size 1.27 1.27)) hide)
     )
-    (property "Value" "DIODE" (id 1) (at 96.012 94.234 0)
+    (property "Value" "LED" (id 1) (at 96.012 94.234 0)
       (effects (font (size 0.762 0.762)))
     )
@@
       (effects (font (size 1.27 1.27)) hide)
     )
-    (property "Value" "15 V Switch" (id 1) (at 119.126 85.852 0)
+    (property "Value" "Ignition Switch" (id 1) (at 119.126 85.852 0)
       (effects (font (size 0.762 0.762)))
     )
@@
       (effects (font (size 1.27 1.27)) hide)
     )
-    (property "Value" "Brake Override" (id 1) (at 97.282 85.852 0)
+    (property "Value" "Brake Over-travel" (id 1) (at 97.282 85.852 0)
       (effects (font (size 0.762 0.762)))
     )

Commit message: Shifting added to DTM Dash
Parts:
- added F?: 1A Fuse, symbol Device:Fuse
- added U?: Shift Up, symbol SCR23 Library:Pushbutton_(Open)
- added U?: Shift Down, symbol SCR23 Library:Pushbutton_(Open)
Connections:
- new net: F?.2, U?., U?.
- new net: D?.1 (A), U?., U?.

Commit message: fix everything
shid
Connections:
- new net: F?.2, U?., U?.
- new net: D?.1 (A), U?., U?.
- now unconnected: U?., U?.

Commit message: Create new top level
Parts:
- D? (x2): value LED -> (none)
- F?: value 1A Fuse -> (none)
- U?: value DTM_Dash -> (none)
- U?: value E_Stop -> (none)
- U?: value Shift Up -> (none)
- U?: value Ignition Switch -> (none)
- U?: value Shift Down -> (none)
- U?: value Start Button -> (none)
- U?: value Brake Over-travel -> (none)
Connections:
- new net: F?.2, U?., U?.
- new net: D?.1 (A), U?., U?.
- now unconnected: U?., U?.
Changed lines of the file:
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@@
       (effects (font (size 1.27 1.27)) hide)
     )
-    (property "Value" "1A Fuse" (id 1) (at 140.208 73.66 90))
+    (property "Value" "" (id 1) (at 140.208 73.66 90))
     (property "Footprint" "" (id 2) (at 140.208 75.946 90)
       (effects (font (size 1.27 1.27)) hide)
@@
       (effects (font (size 1.27 1.27)) (justify left) hide)
     )
-    (property "Value" "DTM_Dash" (id 1) (at 152.908 87.63 0)
+    (property "Value" "" (id 1) (at 152.908 87.63 0)
       (effects (font (size 1.27 1.27)) (justify left) hide)
     )
@@
       (effects (font (size 1.27 1.27)) hide)
     )
-    (property "Value" "E_Stop" (id 1) (at 190.246 83.82 0)
+    (property "Value" "" (id 1) (at 190.246 83.82 0)
       (effects (font (size 0.762 0.762)))
     )
@@
       (effects (font (size 1.27 1.27)) hide)
     )
-    (property "Value" "LED" (id 1) (at 199.39 92.456 0)
+    (property "Value" "" (id 1) (at 199.39 92.456 0)
       (effects (font (size 0.762 0.762)))
     )
@@
       (effects (font (size 1.27 1.27)) hide)
     )
-    (property "Value" "LED" (id 1) (at 177.546 92.202 0)
+    (property "Value" "" (id 1) (at 177.546 92.202 0)
       (effects (font (size 0.762 0.762)))
     )
@@
       (effects (font (size 1.27 1.27)) (justify right) hide)
     )
-    (property "Value" "Shift Up" (id 1) (at 123.19 81.788 90)
+    (property "Value" "" (id 1) (at 123.19 81.788 90)
       (effects (font (size 1.27 1.27)) (justify right))
     )
@@
       (effects (font (size 1.27 1.27)) hide)
     )
-    (property "Value" "Ignition Switch" (id 1) (at 200.66 83.82 0)
+    (property "Value" "" (id 1) (at 200.66 83.82 0)
       (effects (font (size 0.762 0.762)))
     )
@@
       (effects (font (size 1.27 1.27)) (justify right) hide)
     )
-    (property "Value" "Shift Down" (id 1) (at 106.68 82.804 90)
+    (property "Value" "" (id 1) (at 106.68 82.804 90)
       (effects (font (size 1.27 1.27)) (justify right))
     )
@@
       (effects (font (size 1.27 1.27)) (justify left) hide)
     )
-    (property "Value" "Start Button" (id 1) (at 192.278 80.772 0)
+    (property "Value" "" (id 1) (at 192.278 80.772 0)
       (effects (font (size 0.762 0.762)) (justify left))
     )
@@
       (effects (font (size 1.27 1.27)) hide)
     )
-    (property "Value" "Brake Over-travel" (id 1) (at 178.816 83.82 0)
+    (property "Value" "" (id 1) (at 178.816 83.82 0)
       (effects (font (size 0.762 0.762)))
     )
@@
       (effects (font (size 1.27 1.27)) hide)
     )
-    (property "Value" "GND" (id 1) (at 192.532 89.916 90)
+    (property "Value" "" (id 1) (at 192.532 89.916 90)
       (effects (font (size 0.762 0.762)) (justify right))
     )

Commit message: HUGE TOP LEVEL
Parts:
- D? (x2): value (none) -> LED
- F?: value (none) -> 1A Fuse
- U?: value (none) -> DTM_Dash
- U?: value (none) -> E_Stop
- U?: value (none) -> Shift Up
- U?: value (none) -> Ignition Switch
- U?: value (none) -> Shift Down
- U?: value (none) -> Start Button
- U?: value (none) -> Brake Over-travel
Connections:
- new net: F?.2, U?., U?.
- new net: D?.1 (A), U?., U?.
- now unconnected: U?., U?.
Changed lines of the file:
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@@
       (effects (font (size 1.27 1.27)) hide)
     )
-    (property "Value" "" (id 1) (at 140.208 73.66 90))
+    (property "Value" "1A Fuse" (id 1) (at 140.208 73.66 90))
     (property "Footprint" "" (id 2) (at 140.208 75.946 90)
       (effects (font (size 1.27 1.27)) hide)
@@
       (effects (font (size 1.27 1.27)) (justify left) hide)
     )
-    (property "Value" "" (id 1) (at 152.908 87.63 0)
+    (property "Value" "DTM_Dash" (id 1) (at 152.908 87.63 0)
       (effects (font (size 1.27 1.27)) (justify left) hide)
     )
@@
       (effects (font (size 1.27 1.27)) hide)
     )
-    (property "Value" "" (id 1) (at 190.246 83.82 0)
+    (property "Value" "E_Stop" (id 1) (at 190.246 83.82 0)
       (effects (font (size 0.762 0.762)))
     )
@@
       (effects (font (size 1.27 1.27)) hide)
     )
-    (property "Value" "" (id 1) (at 199.39 92.456 0)
+    (property "Value" "LED" (id 1) (at 199.39 92.456 0)
       (effects (font (size 0.762 0.762)))
     )
@@
       (effects (font (size 1.27 1.27)) hide)
     )
-    (property "Value" "" (id 1) (at 177.546 92.202 0)
+    (property "Value" "LED" (id 1) (at 177.546 92.202 0)
       (effects (font (size 0.762 0.762)))
     )
@@
       (effects (font (size 1.27 1.27)) (justify right) hide)
     )
-    (property "Value" "" (id 1) (at 123.19 81.788 90)
+    (property "Value" "Shift Up" (id 1) (at 123.19 81.788 90)
       (effects (font (size 1.27 1.27)) (justify right))
     )
@@
       (effects (font (size 1.27 1.27)) hide)
     )
-    (property "Value" "" (id 1) (at 200.66 83.82 0)
+    (property "Value" "Ignition Switch" (id 1) (at 200.66 83.82 0)
       (effects (font (size 0.762 0.762)))
     )
@@
       (effects (font (size 1.27 1.27)) (justify right) hide)
     )
-    (property "Value" "" (id 1) (at 106.68 82.804 90)
+    (property "Value" "Shift Down" (id 1) (at 106.68 82.804 90)
       (effects (font (size 1.27 1.27)) (justify right))
     )
@@
       (effects (font (size 1.27 1.27)) (justify left) hide)
     )
-    (property "Value" "" (id 1) (at 192.278 80.772 0)
+    (property "Value" "Start Button" (id 1) (at 192.278 80.772 0)
       (effects (font (size 0.762 0.762)) (justify left))
     )
@@
       (effects (font (size 1.27 1.27)) hide)
     )
-    (property "Value" "" (id 1) (at 178.816 83.82 0)
+    (property "Value" "Brake Over-travel" (id 1) (at 178.816 83.82 0)
       (effects (font (size 0.762 0.762)))
     )
@@
       (effects (font (size 1.27 1.27)) hide)
     )
-    (property "Value" "" (id 1) (at 192.532 89.916 90)
+    (property "Value" "GND" (id 1) (at 192.532 89.916 90)
       (effects (font (size 0.762 0.762)) (justify right))
     )

Commit message: Filled in Many Sheets
Connections:
- new net: F?.2, U?., U?.
- new net: D?.1 (A), U?., U?.
- now unconnected: U?., U?.
