File: F22 V2 Wiring Schematic.kicad_sch (KiCad schematic)
At the start: 0 parts

Commit message: Create new top level
Other:
- sheet ECU Pin Schematic renamed ECU
- added sheet Dashboard (Dashboard.kicad_sch)
- added sheet Engine (Engine.kicad_sch)
- added sheet Fuse Box (Fuse Box.kicad_sch)
- sheet ECU: file FuseBox.kicad_sch -> ECU.kicad_sch
Changed lines of the file:
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@@
 (kicad_sch (version 20211123) (generator eeschema)
   (paper "A4")
-  (sheet (at 194.056 44.958) (size 37.338 17.018) (fields_autoplaced)
+  (sheet (at 146.558 50.038) (size 30.226 90.932) (fields_autoplaced)
     (stroke (width 0.1524) (type solid) (color 0 0 0 0))
     (fill (color 0 0 0 0.0000))
-    (property "Sheet name" "ECU Pin Schematic" (id 0) (at 194.056 44.2464 0)
+    (property "Sheet name" "Engine" (id 0) (at 146.558 49.3264 0)
       (effects (font (size 1.27 1.27)) (justify left bottom))
     )
-    (property "Sheet file" "FuseBox.kicad_sch" (id 1) (at 194.056 62.5606 0)
+    (property "Sheet file" "Engine.kicad_sch" (id 1) (at 146.558 141.5546 0)
+      (effects (font (size 1.27 1.27)) (justify left top))
+    )
+  )
+  (sheet (at 105.664 50.038) (size 27.94 90.678) (fields_autoplaced)
+    (stroke (width 0.1524) (type solid) (color 0 0 0 0))
+    (fill (color 0 0 0 0.0000))
+    (property "Sheet name" "Fuse Box" (id 0) (at 105.664 49.3264 0)
+      (effects (font (size 1.27 1.27)) (justify left bottom))
+    )
+    (property "Sheet file" "Fuse Box.kicad_sch" (id 1) (at 105.664 141.3006 0)
+      (effects (font (size 1.27 1.27)) (justify left top))
+    )
+  )
+  (sheet (at 64.262 50.038) (size 25.654 90.932) (fields_autoplaced)
+    (stroke (width 0.1524) (type solid) (color 0 0 0 0))
+    (fill (color 0 0 0 0.0000))
+    (property "Sheet name" "ECU" (id 0) (at 64.262 49.3264 0)
+      (effects (font (size 1.27 1.27)) (justify left bottom))
+    )
+    (property "Sheet file" "ECU.kicad_sch" (id 1) (at 64.262 141.5546 0)
+      (effects (font (size 1.27 1.27)) (justify left top))
+    )
+  )
+  (sheet (at 189.738 50.292) (size 32.258 90.932) (fields_autoplaced)
+    (stroke (width 0.1524) (type solid) (color 0 0 0 0))
+    (fill (color 0 0 0 0.0000))
+    (property "Sheet name" "Dashboard" (id 0) (at 189.738 49.5804 0)
+      (effects (font (size 1.27 1.27)) (justify left bottom))
+    )
+    (property "Sheet file" "Dashboard.kicad_sch" (id 1) (at 189.738 141.8086 0)
       (effects (font (size 1.27 1.27)) (justify left top))
     )
@@
     (path "/" (page "1"))
     (path "/d5e68706-1734-4fd4-8c9d-b165d245e9af" (page "2"))
-    (path "/d5e68706-1734-4fd4-8c9d-b165d245e9af/5fb112e4-6825-45ae-bf54-63d687fee381" (page "3"))
+    (path "/c61ebb53-a6d0-4444-86d9-f19c0fecfdba" (page "3"))
     (path "/d5e68706-1734-4fd4-8c9d-b165d245e9af/53ac2e2d-c2df-4ea2-a089-bbe68ee8714f" (page "4"))
     (path "/d5e68706-1734-4fd4-8c9d-b165d245e9af/7d7721af-ff65-4fec-b227-3953c58d72e6" (page "5"))
     (path "/d5e68706-1734-4fd4-8c9d-b165d245e9af/9497869a-07db-4902-ab45-929f549baad6" (page "6"))
     (path "/d5e68706-1734-4fd4-8c9d-b165d245e9af/7c62c02e-06a1-4b87-9f1e-fbacd6b03153" (page "7"))
-    (path "/d5e68706-1734-4fd4-8c9d-b165d245e9af/1e9ec499-b2d5-4724-ba6d-0e62ea65c89a" (page "8"))
+    (path "/8089b290-d208-4c94-858c-dff9966b58d6" (page "8"))
+    (path "/d75c62e5-497b-4bcb-875e-651ecad01f1b" (page "9"))
   )
   (symbol_instances
@@
       (reference "F?") (unit 1) (value "1A Fuse") (footprint "")
     )
-    (path "/d5e68706-1734-4fd4-8c9d-b165d245e9af/5fb112e4-6825-45ae-bf54-63d687fee381/3693eb7a-dc6e-427e-954b-8fe4aa37f7ca"
+    (path "/c61ebb53-a6d0-4444-86d9-f19c0fecfdba/3693eb7a-dc6e-427e-954b-8fe4aa37f7ca"
       (reference "F?") (unit 1) (value "Fuse 3") (footprint "")
     )
-    (path "/d5e68706-1734-4fd4-8c9d-b165d245e9af/5fb112e4-6825-45ae-bf54-63d687fee381/395d3e01-bff5-4ac7-bd31-10468b55a1ff"
+    (path "/c61ebb53-a6d0-4444-86d9-f19c0fecfdba/395d3e01-bff5-4ac7-bd31-10468b55a1ff"
       (reference "F?") (unit 1) (value "Fuse 1") (footprint "")
     )
-    (path "/d5e68706-1734-4fd4-8c9d-b165d245e9af/5fb112e4-6825-45ae-bf54-63d687fee381/8f47ff78-ca52-4f5b-afa7-9683a8ea3b86"
+    (path "/c61ebb53-a6d0-4444-86d9-f19c0fecfdba/8f47ff78-ca52-4f5b-afa7-9683a8ea3b86"
       (reference "F?") (unit 1) (value "Fuse 4") (footprint "")
     )
@@
       (reference "F?") (unit 1) (value "40AFuse") (footprint "")
     )
-    (path "/d5e68706-1734-4fd4-8c9d-b165d245e9af/5fb112e4-6825-45ae-bf54-63d687fee381/cb22fe25-46a7-40e3-a16c-5ad37b50926c"
+    (path "/c61ebb53-a6d0-4444-86d9-f19c0fecfdba/cb22fe25-46a7-40e3-a16c-5ad37b50926c"
       (reference "F?") (unit 1) (value "Fuse 2") (footprint "")
     )
@@
       (reference "INJ?") (unit 1) (value "L") (footprint "")
     )
-    (path "/d5e68706-1734-4fd4-8c9d-b165d245e9af/5fb112e4-6825-45ae-bf54-63d687fee381/1934fbee-ba19-4311-b371-149caf5afa9e"
+    (path "/c61ebb53-a6d0-4444-86d9-f19c0fecfdba/1934fbee-ba19-4311-b371-149caf5afa9e"
       (reference "K?") (unit 1) (value "Relay") (footprint "")
     )
-    (path "/d5e68706-1734-4fd4-8c9d-b165d245e9af/5fb112e4-6825-45ae-bf54-63d687fee381/634dd138-85c3-4319-9ce6-b1a8d1b05163"
+    (path "/c61ebb53-a6d0-4444-86d9-f19c0fecfdba/634dd138-85c3-4319-9ce6-b1a8d1b05163"
       (reference "K?") (unit 1) (value "Relay") (footprint "")
     )
@@
       (reference "K?") (unit 1) (value "Starter Relay") (footprint "")
     )
-    (path "/d5e68706-1734-4fd4-8c9d-b165d245e9af/5fb112e4-6825-45ae-bf54-63d687fee381/9fb1d08d-a25d-489b-a49c-09206220bcc2"
+    (path "/c61ebb53-a6d0-4444-86d9-f19c0fecfdba/9fb1d08d-a25d-489b-a49c-09206220bcc2"
       (reference "K?") (unit 1) (value "Relay") (footprint "")
     )
-    (path "/d5e68706-1734-4fd4-8c9d-b165d245e9af/5fb112e4-6825-45ae-bf54-63d687fee381/c6eb419e-c626-467b-9e45-ee012504670a"
+    (path "/c61ebb53-a6d0-4444-86d9-f19c0fecfdba/c6eb419e-c626-467b-9e45-ee012504670a"
       (reference "K?") (unit 1) (value "Relay") (footprint "")
     )
@@
       (reference "U?") (unit 1) (value "E_Stop") (footprint "")
     )
-    (path "/d5e68706-1734-4fd4-8c9d-b165d245e9af/5fb112e4-6825-45ae-bf54-63d687fee381/48386ff0-d03e-46fe-bdc6-f35bb77ab890"
+    (path "/c61ebb53-a6d0-4444-86d9-f19c0fecfdba/48386ff0-d03e-46fe-bdc6-f35bb77ab890"
       (reference "U?") (unit 1) (value "DT_12_Pin") (footprint "")
     )
@@
       (reference "U?") (unit 1) (value "ECU2") (footprint "")
     )
-    (path "/d5e68706-1734-4fd4-8c9d-b165d245e9af/5fb112e4-6825-45ae-bf54-63d687fee381/7ca7f5ef-bd73-4f92-b872-9c50ea8c59e3"
+    (path "/c61ebb53-a6d0-4444-86d9-f19c0fecfdba/7ca7f5ef-bd73-4f92-b872-9c50ea8c59e3"
       (reference "U?") (unit 1) (value "Bridge") (footprint "")
-    )
-    (path "/d5e68706-1734-4fd4-8c9d-b165d245e9af/1e9ec499-b2d5-4724-ba6d-0e62ea65c89a/7d654b39-a802-4ca3-b327-07f35da08bc7"
-      (reference "U?") (unit 1) (value "ECU_Engine") (footprint "")
     )
     (path "/d5e68706-1734-4fd4-8c9d-b165d245e9af/9497869a-07db-4902-ab45-929f549baad6/85f93514-dcb0-41b7-96bd-fdec7c68ce6d"
@@
       (reference "U?") (unit 1) (value "Shift Down") (footprint "")
     )
-    (path "/d5e68706-1734-4fd4-8c9d-b165d245e9af/5fb112e4-6825-45ae-bf54-63d687fee381/9ad36b87-025b-4660-a2a7-2295d4ef041a"
+    (path "/c61ebb53-a6d0-4444-86d9-f19c0fecfdba/9ad36b87-025b-4660-a2a7-2295d4ef041a"
       (reference "U?") (unit 1) (value "DTM04-12pb") (footprint "")
     )
@@
       (reference "U?") (unit 1) (value "Start Button") (footprint "")
     )
-    (path "/d5e68706-1734-4fd4-8c9d-b165d245e9af/5fb112e4-6825-45ae-bf54-63d687fee381/c19ff2e9-90b3-4963-ad0e-1db686587abb"
+    (path "/c61ebb53-a6d0-4444-86d9-f19c0fecfdba/c19ff2e9-90b3-4963-ad0e-1db686587abb"
       (reference "U?") (unit 1) (value "Bridge") (footprint "")
     )
-    (path "/d5e68706-1734-4fd4-8c9d-b165d245e9af/1e9ec499-b2d5-4724-ba6d-0e62ea65c89a/c67ae3b5-6133-4d16-9d57-73936b4775aa"
-      (reference "U?") (unit 1) (value "DTM_Engine_Sensors") (footprint "")
-    )
     (path "/d5e68706-1734-4fd4-8c9d-b165d245e9af/53ac2e2d-c2df-4ea2-a089-bbe68ee8714f/d716e568-9167-484a-872e-e4bb0c920da3"

Commit message: HUGE TOP LEVEL
Parts:
- added R? (x2): R120, symbol Device:R
Connections:
- new net CANH: R?.1, R?.1
- new net CANL: R?.2, R?.2
Other:
- added sheet Coil Driver (Coil_Driver.kicad_sch)

Commit message: Getting Ready for CDR
Other:
- removed sheet Coil Driver
Changed lines of the file:
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@@
     (stroke (width 0) (type default) (color 0 0 0 0))
   )
-  (wire (pts (xy 179.324 107.696) (xy 192.532 107.696))
+  (wire (pts (xy 135.89 107.696) (xy 192.532 107.696))
     (stroke (width 0) (type default) (color 0 0 0 0))
   )
@@
     (stroke (width 0) (type default) (color 0 0 0 0))
   )
-  (wire (pts (xy 135.89 113.792) (xy 151.638 113.792))
-    (stroke (width 0) (type default) (color 0 0 0 0))
-  )
   (wire (pts (xy 135.89 62.23) (xy 151.638 62.23))
     (stroke (width 0) (type default) (color 0 0 0 0))
@@
     (stroke (width 0) (type default) (color 0 0 0 0))
   )
-  (wire (pts (xy 179.324 109.728) (xy 192.532 109.728))
+  (wire (pts (xy 135.89 109.728) (xy 192.532 109.728))
     (stroke (width 0) (type default) (color 0 0 0 0))
   )
@@
     (stroke (width 0) (type default) (color 0 0 0 0))
   )
-  (wire (pts (xy 135.89 107.696) (xy 151.638 107.696))
-    (stroke (width 0) (type default) (color 0 0 0 0))
-  )
   (wire (pts (xy 88.646 44.704) (xy 100.33 44.704))
     (stroke (width 0) (type default) (color 0 0 0 0))
@@
     (stroke (width 0) (type default) (color 0 0 0 0))
   )
-  (wire (pts (xy 135.89 109.728) (xy 151.638 109.728))
-    (stroke (width 0) (type default) (color 0 0 0 0))
-  )
   (wire (pts (xy 98.806 52.07) (xy 98.806 37.084))
     (stroke (width 0) (type default) (color 0 0 0 0))
   )
-  (wire (pts (xy 179.324 113.792) (xy 192.532 113.792))
+  (wire (pts (xy 135.89 113.792) (xy 192.532 113.792))
     (stroke (width 0) (type default) (color 0 0 0 0))
   )
@@
     (stroke (width 0) (type default) (color 0 0 0 0))
   )
-  (wire (pts (xy 179.324 111.76) (xy 192.532 111.76))
+  (wire (pts (xy 135.89 111.76) (xy 192.532 111.76))
     (stroke (width 0) (type default) (color 0 0 0 0))
   )
@@
     (stroke (width 0) (type default) (color 0 0 0 0))
   )
-  (wire (pts (xy 135.89 111.76) (xy 151.638 111.76))
-    (stroke (width 0) (type default) (color 0 0 0 0))
-  )
   (wire (pts (xy 135.89 98.806) (xy 192.532 98.806))
     (stroke (width 0) (type default) (color 0 0 0 0))
   )
-  (wire (pts (xy 135.89 115.824) (xy 151.638 115.824))
-    (stroke (width 0) (type default) (color 0 0 0 0))
-  )
   (wire (pts (xy 183.388 55.88) (xy 192.278 55.88))
     (stroke (width 0) (type default) (color 0 0 0 0))
@@
     (effects (font (size 1.27 1.27)) (justify right))
   )
-  (hierarchical_label "COIL_SGN_1" (shape input) (at 135.89 113.792 180)
-    (effects (font (size 1.27 1.27)) (justify right))
-  )
   (hierarchical_label "BAT_FUSE" (shape output) (at 183.388 53.848 180)
     (effects (font (size 1.27 1.27)) (justify right))
   )
-  (hierarchical_label "COIL_SGN_2" (shape input) (at 135.89 111.76 180)
-    (effects (font (size 1.27 1.27)) (justify right))
-  )
-  (hierarchical_label "COIL_1" (shape input) (at 179.324 113.792 180)
+  (hierarchical_label "COIL_1" (shape input) (at 135.89 113.792 180)
     (effects (font (size 1.27 1.27)) (justify right))
   )
@@
     (effects (font (size 1.27 1.27)) (justify right))
   )
-  (hierarchical_label "COIL_SGN_4" (shape input) (at 151.638 107.696 0)
-    (effects (font (size 1.27 1.27)) (justify left))
-  )
-  (hierarchical_label "COIL_3" (shape input) (at 179.324 109.728 180)
+  (hierarchical_label "COIL_3" (shape input) (at 135.89 109.728 180)
     (effects (font (size 1.27 1.27)) (justify right))
   )
@@
     (effects (font (size 1.27 1.27)) (justify left))
   )
-  (hierarchical_label "COIL_4" (shape input) (at 179.324 107.696 180)
+  (hierarchical_label "COIL_4" (shape input) (at 135.89 107.696 180)
     (effects (font (size 1.27 1.27)) (justify right))
   )
@@
     (effects (font (size 1.27 1.27)) (justify right))
   )
-  (hierarchical_label "COIL_GND" (shape input) (at 151.638 115.824 0)
-    (effects (font (size 1.27 1.27)) (justify left))
-  )
   (hierarchical_label "INJ_2" (shape input) (at 135.89 100.838 180)
     (effects (font (size 1.27 1.27)) (justify right))
@@
     (effects (font (size 1.27 1.27)) (justify right))
   )
-  (hierarchical_label "COIL_SGN_3" (shape input) (at 135.89 109.728 180)
-    (effects (font (size 1.27 1.27)) (justify right))
-  )
   (hierarchical_label "COIL_2" (shape input) (at 192.532 111.76 0)
     (effects (font (size 1.27 1.27)) (justify left))
@@
     (effects (font (size 1.27 1.27)) (justify left))
   )
-  (hierarchical_label "COIL_GND" (shape input) (at 135.89 115.824 180)
-    (effects (font (size 1.27 1.27)) (justify right))
-  )
   (hierarchical_label "MAP_SGN" (shape input) (at 135.89 82.55 180)
     (effects (font (size 1.27 1.27)) (justify right))
@@
     (effects (font (size 1.27 1.27)) (justify left))
   )
-  (hierarchical_label "COIL_SGN_3" (shape input) (at 151.638 109.728 0)
-    (effects (font (size 1.27 1.27)) (justify left))
-  )
   (hierarchical_label "IAT" (shape output) (at 135.89 88.646 180)
     (effects (font (size 1.27 1.27)) (justify right))
@@
     (effects (font (size 1.27 1.27)) (justify left))
   )
-  (hierarchical_label "COIL_SGN_1" (shape input) (at 151.638 113.792 0)
-    (effects (font (size 1.27 1.27)) (justify left))
-  )
   (hierarchical_label "IGN_SWITCH" (shape output) (at 110.236 56.134 0)
     (effects (font (size 1.27 1.27)) (justify left))
@@
     (effects (font (size 1.27 1.27)) (justify left))
   )
-  (hierarchical_label "COIL_SGN_4" (shape input) (at 135.89 107.696 180)
-    (effects (font (size 1.27 1.27)) (justify right))
-  )
   (hierarchical_label "IGN_SWITCH" (shape input) (at 97.79 56.134 180)
     (effects (font (size 1.27 1.27)) (justify right))
@@
     (effects (font (size 1.27 1.27)) (justify right))
   )
-  (hierarchical_label "COIL_SGN_2" (shape input) (at 151.638 111.76 0)
-    (effects (font (size 1.27 1.27)) (justify left))
-  )
   (hierarchical_label "IGN_SWITCH" (shape input) (at 135.89 56.134 180)
     (effects (font (size 1.27 1.27)) (justify right))
@@
     (effects (font (size 1.27 1.27)) (justify right))
   )
-  (hierarchical_label "COIL_2" (shape input) (at 179.324 111.76 180)
+  (hierarchical_label "COIL_2" (shape input) (at 135.89 111.76 180)
     (effects (font (size 1.27 1.27)) (justify right))
   )
@@
     )
   )
-  (sheet (at 151.638 106.426) (size 27.94 10.922) (fields_autoplaced)
-    (stroke (width 0.1524) (type solid) (color 0 0 0 0))
-    (fill (color 0 0 0 0.0000))
-    (property "Sheet name" "Coil Driver" (id 0) (at 151.638 105.7144 0)
-      (effects (font (size 1.27 1.27)) (justify left bottom))
-    )
-    (property "Sheet file" "Coil_Driver.kicad_sch" (id 1) (at 151.638 117.9326 0)
-      (effects (font (size 1.27 1.27)) (justify left top))
-    )
-  )
   (sheet (at 110.236 50.292) (size 25.654 93.218) (fields_autoplaced)
     (stroke (width 0.1524) (type solid) (color 0 0 0 0))
@@
     (path "/d5e68706-1734-4fd4-8c9d-b165d245e9af" (page "2"))
     (path "/c61ebb53-a6d0-4444-86d9-f19c0fecfdba" (page "3"))
+    (path "/d5e68706-1734-4fd4-8c9d-b165d245e9af/4de61517-d9cf-4c7a-9bf3-3fb541f362af" (page "4"))
     (path "/d5e68706-1734-4fd4-8c9d-b165d245e9af/03908c32-4728-430d-99d4-f08a90aea921" (page "7"))
     (path "/8089b290-d208-4c94-858c-dff9966b58d6" (page "8"))
     (path "/d75c62e5-497b-4bcb-875e-651ecad01f1b" (page "9"))
-    (path "/cd87b180-e5e1-4fae-8636-4859bb94d6e9" (page "10"))
   )
   (symbol_instances
