File: Coil_Driver.kicad_sch (KiCad schematic)
At the start: 0 parts

Commit message: Filled in Many Sheets
Other:
- note added: "Go Back Up Stupid"
Changed lines of the file:
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@@
 (kicad_sch (version 20211123) (generator eeschema)
   (paper "A4")
+  (text "Go Back Up Stupid" (at 130.048 88.646 0)
+    (effects (font (size 2.54 2.54)) (justify left bottom))
+  )
 )
