File: Dashboard.kicad_sch (KiCad schematic)
At the start: 11 parts

Commit message: readd all connectors
Parts:
- D? (x2): value LED -> ${SIM.PARAMS}; Spice_Netlist_Enabled Y -> (none); Spice_Primitive D -> (none)
Connections:
- new net: D?.1 (A), U?., U?.
- new net: F?.2, U?., U?.
- now unconnected: U?., U?.

Commit message: Updating Connectors
Connections:
- new net: D?.1 (A), U?., U?.
- new net: F?.2, U?., U?.
- now unconnected: U?., U?.
