File: Engine.kicad_sch (KiCad schematic)
At the start: 16 parts

Commit message: readd all connectors
Parts:
- U?: value DT_12P_Green_Male - 20 -> DT_12P_Green_Male - #20
- U?: value DTM_12P_Green_Male - 19 -> DTM_12P_Green_Male - #19
